Commit message: fix: restore official MechArm visuals and joint controller

File: tak2/ros2_ws/src/task2_sim/urdf/mecharm_270_gazebo.urdf (robot description, URDF)
Before this commit: robot mecharm_270_gazebo, 7 links, 6 joints
Links:
- link base: geometry collision mesh filename=package://mycobot_description/urdf/mecharm_270_m5/base.dae; visual mesh filename=package://mycobot_description/urdf/mecharm_270_m5/base.dae
- link link1: geometry collision mesh filename=package://mycobot_description/urdf/mecharm_270_m5/link1.dae; visual mesh filename=package://mycobot_description/urdf/mecharm_270_m5/link1.dae
- link link2: geometry collision mesh filename=package://mycobot_description/urdf/mecharm_270_m5/link2.dae; visual mesh filename=package://mycobot_description/urdf/mecharm_270_m5/link2.dae
- link link3: geometry collision mesh filename=package://mycobot_description/urdf/mecharm_270_m5/link3.dae; visual mesh filename=package://mycobot_description/urdf/mecharm_270_m5/link3.dae
- link link4: geometry collision mesh filename=package://mycobot_description/urdf/mecharm_270_m5/link4.dae; visual mesh filename=package://mycobot_description/urdf/mecharm_270_m5/link4.dae
- link link5: geometry collision mesh filename=package://mycobot_description/urdf/mecharm_270_m5/link5.dae; visual mesh filename=package://mycobot_description/urdf/mecharm_270_m5/link5.dae
- link link6: geometry collision mesh filename=package://mycobot_description/urdf/mecharm_270_m5/link6.dae; visual mesh filename=package://mycobot_description/urdf/mecharm_270_m5/link6.dae
Joints:
- joint joint1_to_base: limit lower=-2.792527 upper=2.792527 effort=20.0 velocity=1.5 -> lower=-2.792527 upper=2.792527 effort=1000.0 velocity=1.5
- joint joint2_to_joint1: limit lower=-1.3089 upper=2.0943 effort=20.0 velocity=1.5 -> lower=-1.3089 upper=2.0943 effort=1000.0 velocity=1.5; origin xyz=0 0 0.038 rpy=-1.5708 0 0 -> xyz=0 0 0.038 rpy= -1.5708 0 0 
- joint joint3_to_joint2: axis 0 0 1 ->  0 0 1; limit lower=-3.0543 upper=1.1344 effort=20.0 velocity=1.5 -> lower=-3.0543 upper=1.1344 effort=1000.0 velocity=1.5; origin xyz=0 -0.1 0 rpy=0 0 0 -> xyz=0.0 -0.1 0    rpy=0 0 0 
- joint joint4_to_joint3: axis 0 0 1 ->  0 0 1; limit lower=-2.7052 upper=2.7052 effort=15.0 velocity=1.5 -> lower=-2.7052 upper=2.7052 effort=1000.0 velocity=1.5; origin xyz=0.108 -0.005 -0.001 rpy=0 1.5708 0 -> xyz=0.108 -0.005  -0.001 rpy=0 1.5708 0 
- joint joint5_to_joint4: limit lower=-2.0071 upper=2.0071 effort=12.0 velocity=1.5 -> lower=-2.0071 upper=2.0071 effort=1000.0 velocity=1.5; origin xyz=-0.001 0 0 rpy=0 -1.5708 0 -> xyz= -0.001 0 0.0 rpy=  0 -1.5708 0
- joint joint6_to_joint5: limit lower=-3.14 upper=3.14 effort=10.0 velocity=1.5 -> lower=-3.14 upper=3.14 effort=1000.0 velocity=1.5; origin xyz=0.06 0 0 rpy=0 1.5708 0 -> xyz= 0.06 0.00 -0.0 rpy=  0 1.5708 0 

Commit message: fix: anchor robot base and smooth joint motion

File: tak2/ros2_ws/src/task2_sim/urdf/mecharm_270_gazebo.urdf (robot description, URDF)
Before this commit: robot firefighter, 7 links, 6 joints
Links:
- added link world
Joints:
- added joint world_fixed: type fixed, parent world, child base, origin xyz=0 0 0 rpy=0 0 0

Commit message: feat: add physical two-finger gripper for pick and place

File: tak2/ros2_ws/src/task2_sim/urdf/mecharm_270_gazebo.urdf (robot description, URDF)
Before this commit: robot firefighter, 8 links, 7 joints
Links:
- added link gripper_palm, mass 0.08; collision box size=0.078 0.026 0.015; visual box size=0.078 0.026 0.015
- added link left_finger, mass 0.025; collision box size=0.008 0.014 0.055; visual box size=0.008 0.014 0.055
- added link right_finger, mass 0.025; collision box size=0.008 0.014 0.055; visual box size=0.008 0.014 0.055
Joints:
- added joint gripper_mount: type fixed, parent link6, child gripper_palm, origin xyz=0 0 0.005 rpy=0 0 0
- added joint left_finger_joint: type prismatic, parent gripper_palm, child left_finger, origin xyz=0.035 0 0.015 rpy=0 0 0, axis -1 0 0, limit lower=0.0 upper=0.010 effort=30 velocity=0.04
- added joint right_finger_joint: type prismatic, parent gripper_palm, child right_finger, origin xyz=-0.035 0 0.015 rpy=0 0 0, axis 1 0 0, limit lower=0.0 upper=0.010 effort=30 velocity=0.04

Commit message: fix: increase gripper force and contact friction

File: tak2/ros2_ws/src/task2_sim/urdf/mecharm_270_gazebo.urdf (robot description, URDF)
Before this commit: robot firefighter, 11 links, 10 joints
Joints:
- joint left_finger_joint: limit lower=0.0 upper=0.010 effort=30 velocity=0.04 -> lower=0.0 upper=0.010 effort=60 velocity=0.04
- joint right_finger_joint: limit lower=0.0 upper=0.010 effort=30 velocity=0.04 -> lower=0.0 upper=0.010 effort=60 velocity=0.04

Commit message: fix: stabilize physical grasp and precise placement

File: tak2/ros2_ws/src/task2_sim/urdf/mecharm_270_gazebo.urdf (robot description, URDF)
Before this commit: robot firefighter, 11 links, 10 joints
Links:
- link left_finger: geometry collision box size=0.010 0.026 0.048; visual box size=0.010 0.026 0.048
- link right_finger: geometry collision box size=0.010 0.026 0.048; visual box size=0.010 0.026 0.048
Joints:
- joint joint1_to_base: limit lower=-2.792527 upper=2.792527 effort=1000.0 velocity=1.5 -> lower=-2.792527 upper=2.792527 effort=20.0 velocity=1.5
- joint joint2_to_joint1: limit lower=-1.3089 upper=2.0943 effort=1000.0 velocity=1.5 -> lower=-1.3089 upper=2.0943 effort=25.0 velocity=1.5
- joint joint3_to_joint2: limit lower=-3.0543 upper=1.1344 effort=1000.0 velocity=1.5 -> lower=-3.0543 upper=1.1344 effort=22.0 velocity=1.5
- joint joint4_to_joint3: limit lower=-2.7052 upper=2.7052 effort=1000.0 velocity=1.5 -> lower=-2.7052 upper=2.7052 effort=12.0 velocity=1.5
- joint joint5_to_joint4: limit lower=-2.0071 upper=2.0071 effort=1000.0 velocity=1.5 -> lower=-2.0071 upper=2.0071 effort=10.0 velocity=1.5
- joint joint6_to_joint5: limit lower=-3.14 upper=3.14 effort=1000.0 velocity=1.5 -> lower=-3.14 upper=3.14 effort=8.0 velocity=1.5
- joint left_finger_joint: limit lower=0.0 upper=0.010 effort=60 velocity=0.04 -> lower=0.0 upper=0.010 effort=20 velocity=0.04
- joint right_finger_joint: limit lower=0.0 upper=0.010 effort=60 velocity=0.04 -> lower=0.0 upper=0.010 effort=20 velocity=0.04

Commit message: fix: restore proven stable arm control and placement margin

File: tak2/ros2_ws/src/task2_sim/urdf/mecharm_270_gazebo.urdf (robot description, URDF)
Before this commit: robot firefighter, 11 links, 10 joints
Joints:
- joint joint1_to_base: limit lower=-2.792527 upper=2.792527 effort=20.0 velocity=1.5 -> lower=-2.792527 upper=2.792527 effort=1000.0 velocity=1.5
- joint joint2_to_joint1: limit lower=-1.3089 upper=2.0943 effort=25.0 velocity=1.5 -> lower=-1.3089 upper=2.0943 effort=1000.0 velocity=1.5
- joint joint3_to_joint2: limit lower=-3.0543 upper=1.1344 effort=22.0 velocity=1.5 -> lower=-3.0543 upper=1.1344 effort=1000.0 velocity=1.5
- joint joint4_to_joint3: limit lower=-2.7052 upper=2.7052 effort=12.0 velocity=1.5 -> lower=-2.7052 upper=2.7052 effort=1000.0 velocity=1.5
- joint joint5_to_joint4: limit lower=-2.0071 upper=2.0071 effort=10.0 velocity=1.5 -> lower=-2.0071 upper=2.0071 effort=1000.0 velocity=1.5
- joint joint6_to_joint5: limit lower=-3.14 upper=3.14 effort=8.0 velocity=1.5 -> lower=-3.14 upper=3.14 effort=1000.0 velocity=1.5

Commit message: fix: restore proven stable arm and gripper baseline

File: tak2/ros2_ws/src/task2_sim/urdf/mecharm_270_gazebo.urdf (robot description, URDF)
Before this commit: robot firefighter, 11 links, 10 joints
Links:
- link left_finger: geometry collision box size=0.008 0.014 0.055; visual box size=0.008 0.014 0.055
- link right_finger: geometry collision box size=0.008 0.014 0.055; visual box size=0.008 0.014 0.055
Joints:
- joint left_finger_joint: limit lower=0.0 upper=0.010 effort=20 velocity=0.04 -> lower=0.0 upper=0.010 effort=60 velocity=0.04
- joint right_finger_joint: limit lower=0.0 upper=0.010 effort=20 velocity=0.04 -> lower=0.0 upper=0.010 effort=60 velocity=0.04

Commit message: fix: align simulation with mechArm 270 Pi adaptive gripper

File: tak2/ros2_ws/src/task2_sim/urdf/mecharm_270_gazebo.urdf (robot description, URDF)
Before this commit: robot firefighter, 11 links, 10 joints
Links:
- link gripper_palm: mass 0.08 -> 0.05
Joints:
- joint left_finger_joint: limit lower=0.0 upper=0.010 effort=60 velocity=0.04 -> lower=0.0 upper=0.0125 effort=60 velocity=0.04; origin xyz=0.035 0 0.015 rpy=0 0 0 -> xyz=0.0265 0 0.015 rpy=0 0 0
- joint right_finger_joint: limit lower=0.0 upper=0.010 effort=60 velocity=0.04 -> lower=0.0 upper=0.0125 effort=60 velocity=0.04; origin xyz=-0.035 0 0.015 rpy=0 0 0 -> xyz=-0.0265 0 0.015 rpy=0 0 0

Commit message: feat: model adaptive gripper linkage for simulation

File: tak2/ros2_ws/src/task2_sim/urdf/mecharm_270_gazebo.urdf (robot description, URDF)
Before this commit: robot mecharm_270_pi, 11 links, 10 joints
Links:
- removed link left_finger
- removed link right_finger
- added link gripper_left1, mass 0.018; collision box size=0.010 0.022 0.030; visual box size=0.004 0.024 0.030
- added link gripper_left2, mass 0.010; collision box size=0.030 0.008 0.008; visual box size=0.030 0.008 0.008
- added link gripper_left3, mass 0.012; collision box size=0.008 0.010 0.0315; visual box size=0.008 0.010 0.0315
- added link gripper_right1, mass 0.018; collision box size=0.010 0.022 0.030; visual box size=0.004 0.024 0.030
- added link gripper_right2, mass 0.010; collision box size=0.030 0.008 0.008; visual box size=0.030 0.008 0.008
- added link gripper_right3, mass 0.012; collision box size=0.008 0.010 0.0315; visual box size=0.008 0.010 0.0315
- link gripper_palm: mass 0.05 -> 0.090; geometry collision box size=0.062 0.050 0.026; visual box size=0.065 0.055 0.030
Joints:
- removed joint left_finger_joint
- removed joint right_finger_joint
- added joint gripper_base_to_gripper_left2: type revolute, parent gripper_palm, child gripper_left2, origin xyz=-0.005 0 0.027 rpy=0 0 0, axis 0 -1 0, limit lower=-0.80 upper=0.50 effort=8.0 velocity=1.2
- added joint gripper_base_to_gripper_right2: type revolute, parent gripper_palm, child gripper_right2, origin xyz=0.005 0 0.027 rpy=0 0 0, axis 0 -1 0, limit lower=-0.50 upper=0.80 effort=8.0 velocity=1.2
- added joint gripper_base_to_gripper_right3: type revolute, parent gripper_palm, child gripper_right3, origin xyz=0.012 0 0.005 rpy=0 0 0, axis 0 -1 0, limit lower=-0.15 upper=0.70 effort=8.0 velocity=1.2
- added joint gripper_controller: type revolute, parent gripper_palm, child gripper_left3, origin xyz=-0.012 0 0.005 rpy=0 0 0, axis 0 -1 0, limit lower=-0.70 upper=0.15 effort=8.0 velocity=1.2
- added joint gripper_left3_to_gripper_left1: type revolute, parent gripper_left3, child gripper_left1, origin xyz=-0.027 0 0.016 rpy=0 0 0, axis 0 -1 0, limit lower=-0.50 upper=0.50 effort=8.0 velocity=1.2
- added joint gripper_right3_to_gripper_right1: type revolute, parent gripper_right3, child gripper_right1, origin xyz=0.027 0 0.016 rpy=0 0 0, axis 0 -1 0, limit lower=-0.50 upper=0.50 effort=8.0 velocity=1.2

Commit message: fix: align placement acceptance and gripper pad contact

File: tak2/ros2_ws/src/task2_sim/urdf/mecharm_270_gazebo.urdf (robot description, URDF)
Before this commit: robot mecharm_270_pi, 15 links, 14 joints
Links:
- link gripper_left1: geometry collision box size=0.006 0.030 0.034; collision box size=0.010 0.022 0.030
- link gripper_right1: geometry collision box size=0.006 0.030 0.034; collision box size=0.010 0.022 0.030
