Commit message: fix: tighten grasp to reduce block slip during lift
Diagnosed the block slipping/falling during pick-up as a loose grip
(pad faces ~2 mm wider than the 25 mm object). Slow the descent/lift,
raise block friction and contact damping, close the gripper harder,
and widen the finger-linkage joint limits so the pads can reach the
object. Grasp and placement now verify consistently.

File: task3/ros2_ws/src/task3_sim/urdf/mecharm_270_gazebo.urdf (robot description, URDF)
Before this commit: robot mecharm_270_pi, 15 links, 14 joints
Joints:
- joint gripper_left3_to_gripper_left1: limit lower=-0.50 upper=0.50 effort=8.0 velocity=1.2 -> lower=-0.70 upper=0.70 effort=8.0 velocity=1.2
- joint gripper_right3_to_gripper_right1: limit lower=-0.50 upper=0.50 effort=8.0 velocity=1.2 -> lower=-0.70 upper=0.70 effort=8.0 velocity=1.2
